File: Eco robot/1.1.1/main.sch (EAGLE design)
At the start: 109 parts, among them IC1 REGULATERLM1058, IC2 REGULATERLM1058, Q1 CRYSTALNX5032GA, SW1 SWITCH_4PALPS, SW2 SWITCH_4PALPS, U1 FT232RL, X2 MINI-USB-SHIELD-UX60A-MB-5ST

Commit message: eco new
Connections:
- net VDD: now also U$4G$1.P$2, U$4G$2.P$2
Changed lines of the file:
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@@
 <wire x1="165.1" y1="66.04" x2="167.64" y2="66.04" width="0.1524" layer="91"/>
 <wire x1="167.64" y1="66.04" x2="167.64" y2="60.96" width="0.1524" layer="91"/>
-<wire x1="167.64" y1="60.96" x2="167.64" y2="55.88" width="0.1524" layer="91"/>
+<wire x1="167.64" y1="60.96" x2="167.64" y2="58.42" width="0.1524" layer="91"/>
+<wire x1="167.64" y1="58.42" x2="167.64" y2="55.88" width="0.1524" layer="91"/>
 <wire x1="167.64" y1="55.88" x2="165.1" y2="55.88" width="0.1524" layer="91"/>
 <pinref part="SUPPLY54" gate="G$1" pin="VDD"/>
@@
 <pinref part="U$4" gate="G$1" pin="P$3"/>
 <pinref part="U$4" gate="G$2" pin="P$3"/>
+<pinref part="U$4" gate="G$1" pin="P$2"/>
+<wire x1="157.48" y1="60.96" x2="157.48" y2="58.42" width="0.1524" layer="91"/>
+<wire x1="157.48" y1="58.42" x2="167.64" y2="58.42" width="0.1524" layer="91"/>
+<junction x="167.64" y="58.42"/>
+<pinref part="U$4" gate="G$2" pin="P$2"/>
+<wire x1="157.48" y1="50.8" x2="157.48" y2="48.26" width="0.1524" layer="91"/>
+<wire x1="157.48" y1="48.26" x2="167.64" y2="48.26" width="0.1524" layer="91"/>
+<wire x1="167.64" y1="48.26" x2="167.64" y2="55.88" width="0.1524" layer="91"/>
+<junction x="167.64" y="55.88"/>
 </segment>
 <segment>
